File: breakout_boards/motherboard_extension_board.sch (KiCad schematic (older format))
At the start: 41 parts, among them J1 XM, J10 BLTouch, J11 FAN1, J12 HE1, J13 THE1, J14 ZM1, J15 FAN2, J16 HE2, J17 THE2, J18 ZM2, J19 TFT, J2 NeoPixel, J20 EXP2, J21 EM0, J22 E0-Stop, J23 X-Stop, J24 EM1, J25 E1-Stop, J26 Y-Stop, J27 I2C, J28 EM2, J29 E2-Stop, J3 BED, J30 Z-Stop, J31 Power, J32 5V_PSU, J33 UART, J34 POWER_EXP, J35 SPI, J36 Extension1, J37 Extension2, J4 THB, J5 FAN0, J6 EXP1, J7 YM, J8 HE0, J9 THE0

Commit message: changed mounting hole footprint and connector jst eh to jst xh
Parts:
- H1, H2, H3, H4: footprint MountingHole:MountingHole_3.2mm_M3 -> MountingHole:MountingHole_3.2mm_M3_DIN965
- J1, J14, J18, J21, J24, J27, J28, J33, J7: footprint Connector_JST:JST_EH_B4B-EH-A_1x04_P2.50mm_Vertical -> Connector_JST:JST_XH_B4B-XH-A_1x04_P2.50mm_Vertical
- J10, J19: footprint Connector_JST:JST_EH_B5B-EH-A_1x05_P2.50mm_Vertical -> Connector_JST:JST_XH_B5B-XH-A_1x05_P2.50mm_Vertical
- J11, J12, J13, J15, J16, J17, J3, J4, J5, J8, J9: footprint Connector_JST:JST_EH_B2B-EH-A_1x02_P2.50mm_Vertical -> Connector_JST:JST_XH_B2B-XH-A_1x02_P2.50mm_Vertical
- J22, J23, J25, J26, J29, J30: footprint Connector_JST:JST_EH_B3B-EH-A_1x03_P2.50mm_Vertical -> Connector_JST:JST_XH_B3B-XH-A_1x03_P2.50mm_Vertical
- J35: footprint Connector_JST:JST_EH_B6B-EH-A_1x06_P2.50mm_Vertical -> Connector_JST:JST_XH_B6B-XH-A_1x06_P2.50mm_Vertical
Changed lines of the file:
@@
 F 0 "J4" V 1350 4650 50  0000 L CNN
 F 1 "THB" V 1450 4850 50  0000 L CNN
-F 2 "Connector_JST:JST_EH_B2B-EH-A_1x02_P2.50mm_Vertical" H 1350 4950 50  0001 C CNN
+F 2 "Connector_JST:JST_XH_B2B-XH-A_1x02_P2.50mm_Vertical" H 1350 4950 50  0001 C CNN
 F 3 "~" H 1350 4950 50  0001 C CNN
 	1    1350 4950
@@
 F 0 "J33" H 5018 2825 50  0000 C CNN
 F 1 "UART" H 5018 2916 50  0000 C CNN
-F 2 "Connector_JST:JST_EH_B4B-EH-A_1x04_P2.50mm_Vertical" H 5100 3250 50  0001 C CNN
+F 2 "Connector_JST:JST_XH_B4B-XH-A_1x04_P2.50mm_Vertical" H 5100 3250 50  0001 C CNN
 F 3 "~" H 5100 3250 50  0001 C CNN
 	1    5100 3250
@@
 F 0 "J10" H 1918 3617 50  0000 C CNN
 F 1 "BLTouch" H 1918 3526 50  0000 C CNN
-F 2 "Connector_JST:JST_EH_B5B-EH-A_1x05_P2.50mm_Vertical" H 2000 3200 50  0001 C CNN
+F 2 "Connector_JST:JST_XH_B5B-XH-A_1x05_P2.50mm_Vertical" H 2000 3200 50  0001 C CNN
 F 3 "~" H 2000 3200 50  0001 C CNN
 	1    2000 3200
@@
 F 0 "H4" H 6300 6046 50  0000 L CNN
 F 1 "MountingHole" H 6300 5955 50  0000 L CNN
-F 2 "MountingHole:MountingHole_3.2mm_M3" H 6200 6000 50  0001 C CNN
+F 2 "MountingHole:MountingHole_3.2mm_M3_DIN965" H 6200 6000 50  0001 C CNN
 F 3 "~" H 6200 6000 50  0001 C CNN
 	1    6200 6000
@@
 F 0 "J35" H 5918 2775 50  0000 C CNN
 F 1 "SPI" H 5918 2866 50  0000 C CNN
-F 2 "Connector_JST:JST_EH_B6B-EH-A_1x06_P2.50mm_Vertical" H 6000 3300 50  0001 C CNN
+F 2 "Connector_JST:JST_XH_B6B-XH-A_1x06_P2.50mm_Vertical" H 6000 3300 50  0001 C CNN
 F 3 "~" H 6000 3300 50  0001 C CNN
 	1    6000 3300
@@
 F 0 "J27" H 4018 2825 50  0000 C CNN
 F 1 "I2C" H 4018 2916 50  0000 C CNN
-F 2 "Connector_JST:JST_EH_B4B-EH-A_1x04_P2.50mm_Vertical" H 4100 3250 50  0001 C CNN
+F 2 "Connector_JST:JST_XH_B4B-XH-A_1x04_P2.50mm_Vertical" H 4100 3250 50  0001 C CNN
 F 3 "~" H 4100 3250 50  0001 C CNN
 	1    4100 3250
@@
 F 0 "J28" V 4350 850 50  0000 R CNN
 F 1 "EM2" V 4350 1050 50  0000 R CNN
-F 2 "Connector_JST:JST_EH_B4B-EH-A_1x04_P2.50mm_Vertical" H 4250 950 50  0001 C CNN
+F 2 "Connector_JST:JST_XH_B4B-XH-A_1x04_P2.50mm_Vertical" H 4250 950 50  0001 C CNN
 F 3 "~" H 4250 950 50  0001 C CNN
 	1    4250 950
@@
 F 0 "J24" V 3850 850 50  0000 R CNN
 F 1 "EM1" V 3850 1050 50  0000 R CNN
-F 2 "Connector_JST:JST_EH_B4B-EH-A_1x04_P2.50mm_Vertical" H 3750 950 50  0001 C CNN
+F 2 "Connector_JST:JST_XH_B4B-XH-A_1x04_P2.50mm_Vertical" H 3750 950 50  0001 C CNN
 F 3 "~" H 3750 950 50  0001 C CNN
 	1    3750 950
@@
 F 0 "J19" H 3068 2775 50  0000 C CNN
 F 1 "TFT" H 3068 2866 50  0000 C CNN
-F 2 "Connector_JST:JST_EH_B5B-EH-A_1x05_P2.50mm_Vertical" H 3150 3200 50  0001 C CNN
+F 2 "Connector_JST:JST_XH_B5B-XH-A_1x05_P2.50mm_Vertical" H 3150 3200 50  0001 C CNN
 F 3 "~" H 3150 3200 50  0001 C CNN
 	1    3150 3200
@@
 F 0 "J29" V 4214 3962 50  0000 R CNN
 F 1 "E2-Stop" V 4350 4300 50  0000 R CNN
-F 2 "Connector_JST:JST_EH_B3B-EH-A_1x03_P2.50mm_Vertical" H 4250 4150 50  0001 C CNN
+F 2 "Connector_JST:JST_XH_B3B-XH-A_1x03_P2.50mm_Vertical" H 4250 4150 50  0001 C CNN
 F 3 "~" H 4250 4150 50  0001 C CNN
 	1    4250 4150
@@
 F 0 "J25" V 3714 3962 50  0000 R CNN
 F 1 "E1-Stop" V 3850 4300 50  0000 R CNN
-F 2 "Connector_JST:JST_EH_B3B-EH-A_1x03_P2.50mm_Vertical" H 3750 4150 50  0001 C CNN
+F 2 "Connector_JST:JST_XH_B3B-XH-A_1x03_P2.50mm_Vertical" H 3750 4150 50  0001 C CNN
 F 3 "~" H 3750 4150 50  0001 C CNN
 	1    3750 4150
@@
 F 0 "J16" V 2600 3850 50  0000 L CNN
 F 1 "HE2" V 2700 4050 50  0000 L CNN
-F 2 "Connector_JST:JST_EH_B2B-EH-A_1x02_P2.50mm_Vertical" H 2600 4150 50  0001 C CNN
+F 2 "Connector_JST:JST_XH_B2B-XH-A_1x02_P2.50mm_Vertical" H 2600 4150 50  0001 C CNN
 F 3 "~" H 2600 4150 50  0001 C CNN
 	1    2600 4150
@@
 F 0 "J17" V 2600 4650 50  0000 L CNN
 F 1 "THE2" V 2700 4800 50  0000 L CNN
-F 2 "Connector_JST:JST_EH_B2B-EH-A_1x02_P2.50mm_Vertical" H 2600 4950 50  0001 C CNN
+F 2 "Connector_JST:JST_XH_B2B-XH-A_1x02_P2.50mm_Vertical" H 2600 4950 50  0001 C CNN
 F 3 "~" H 2600 4950 50  0001 C CNN
 	1    2600 4950
@@
 F 0 "J12" V 2200 3850 50  0000 L CNN
 F 1 "HE1" V 2300 4050 50  0000 L CNN
-F 2 "Connector_JST:JST_EH_B2B-EH-A_1x02_P2.50mm_Vertical" H 2200 4150 50  0001 C CNN
+F 2 "Connector_JST:JST_XH_B2B-XH-A_1x02_P2.50mm_Vertical" H 2200 4150 50  0001 C CNN
 F 3 "~" H 2200 4150 50  0001 C CNN
 	1    2200 4150
@@
 F 0 "J13" V 2200 4650 50  0000 L CNN
 F 1 "THE1" V 2300 4800 50  0000 L CNN
-F 2 "Connector_JST:JST_EH_B2B-EH-A_1x02_P2.50mm_Vertical" H 2200 4950 50  0001 C CNN
+F 2 "Connector_JST:JST_XH_B2B-XH-A_1x02_P2.50mm_Vertical" H 2200 4950 50  0001 C CNN
 F 3 "~" H 2200 4950 50  0001 C CNN
 	1    2200 4950
@@
 F 0 "J15" V 2400 5700 50  0000 L CNN
 F 1 "FAN2" V 2500 5850 50  0000 L CNN
-F 2 "Connector_JST:JST_EH_B2B-EH-A_1x02_P2.50mm_Vertical" H 2400 6000 50  0001 C CNN
+F 2 "Connector_JST:JST_XH_B2B-XH-A_1x02_P2.50mm_Vertical" H 2400 6000 50  0001 C CNN
 F 3 "~" H 2400 6000 50  0001 C CNN
 	1    2400 6000
@@
 F 0 "J11" V 2000 5700 50  0000 L CNN
 F 1 "FAN1" V 2100 5850 50  0000 L CNN
-F 2 "Connector_JST:JST_EH_B2B-EH-A_1x02_P2.50mm_Vertical" H 2000 6000 50  0001 C CNN
+F 2 "Connector_JST:JST_XH_B2B-XH-A_1x02_P2.50mm_Vertical" H 2000 6000 50  0001 C CNN
 F 3 "~" H 2000 6000 50  0001 C CNN
 	1    2000 6000
@@
 F 0 "H3" H 6300 5796 50  0000 L CNN
 F 1 "MountingHole" H 6300 5705 50  0000 L CNN
-F 2 "MountingHole:MountingHole_3.2mm_M3" H 6200 5750 50  0001 C CNN
+F 2 "MountingHole:MountingHole_3.2mm_M3_DIN965" H 6200 5750 50  0001 C CNN
 F 3 "~" H 6200 5750 50  0001 C CNN
 	1    6200 5750
@@
 F 0 "H2" H 6300 5546 50  0000 L CNN
 F 1 "MountingHole" H 6300 5455 50  0000 L CNN
-F 2 "MountingHole:MountingHole_3.2mm_M3" H 6200 5500 50  0001 C CNN
+F 2 "MountingHole:MountingHole_3.2mm_M3_DIN965" H 6200 5500 50  0001 C CNN
 F 3 "~" H 6200 5500 50  0001 C CNN
 	1    6200 5500
@@
 F 0 "H1" H 6300 5296 50  0000 L CNN
 F 1 "MountingHole" H 6300 5205 50  0000 L CNN
-F 2 "MountingHole:MountingHole_3.2mm_M3" H 6200 5250 50  0001 C CNN
+F 2 "MountingHole:MountingHole_3.2mm_M3_DIN965" H 6200 5250 50  0001 C CNN
 F 3 "~" H 6200 5250 50  0001 C CNN
 	1    6200 5250
@@
 F 0 "J8" V 1800 3850 50  0000 L CNN
 F 1 "HE0" V 1900 4050 50  0000 L CNN
-F 2 "Connector_JST:JST_EH_B2B-EH-A_1x02_P2.50mm_Vertical" H 1800 4150 50  0001 C CNN
+F 2 "Connector_JST:JST_XH_B2B-XH-A_1x02_P2.50mm_Vertical" H 1800 4150 50  0001 C CNN
 F 3 "~" H 1800 4150 50  0001 C CNN
 	1    1800 4150
@@
 F 0 "J3" V 1350 3850 50  0000 L CNN
 F 1 "BED" V 1450 4000 50  0000 L CNN
-F 2 "Connector_JST:JST_EH_B2B-EH-A_1x02_P2.50mm_Vertical" H 1350 4150 50  0001 C CNN
+F 2 "Connector_JST:JST_XH_B2B-XH-A_1x02_P2.50mm_Vertical" H 1350 4150 50  0001 C CNN
 F 3 "~" H 1350 4150 50  0001 C CNN
 	1    1350 4150
@@
 F 0 "J1" V 1350 800 50  0000 L CNN
 F 1 "XM" V 1350 900 50  0000 L CNN
-F 2 "Connector_JST:JST_EH_B4B-EH-A_1x04_P2.50mm_Vertical" H 1250 950 50  0001 C CNN
+F 2 "Connector_JST:JST_XH_B4B-XH-A_1x04_P2.50mm_Vertical" H 1250 950 50  0001 C CNN
 F 3 "~" H 1250 950 50  0001 C CNN
 	1    1250 950
@@
 F 0 "J18" V 2850 800 50  0000 L CNN
 F 1 "ZM2" V 2850 950 50  0000 L CNN
-F 2 "Connector_JST:JST_EH_B4B-EH-A_1x04_P2.50mm_Vertical" H 2750 950 50  0001 C CNN
+F 2 "Connector_JST:JST_XH_B4B-XH-A_1x04_P2.50mm_Vertical" H 2750 950 50  0001 C CNN
 F 3 "~" H 2750 950 50  0001 C CNN
 	1    2750 950
@@
 F 0 "J22" V 3214 3962 50  0000 R CNN
 F 1 "E0-Stop" V 3350 4300 50  0000 R CNN
-F 2 "Connector_JST:JST_EH_B3B-EH-A_1x03_P2.50mm_Vertical" H 3250 4150 50  0001 C CNN
+F 2 "Connector_JST:JST_XH_B3B-XH-A_1x03_P2.50mm_Vertical" H 3250 4150 50  0001 C CNN
 F 3 "~" H 3250 4150 50  0001 C CNN
 	1    3250 4150
@@
 F 0 "J9" V 1800 4650 50  0000 L CNN
 F 1 "THE0" V 1900 4800 50  0000 L CNN
-F 2 "Connector_JST:JST_EH_B2B-EH-A_1x02_P2.50mm_Vertical" H 1800 4950 50  0001 C CNN
+F 2 "Connector_JST:JST_XH_B2B-XH-A_1x02_P2.50mm_Vertical" H 1800 4950 50  0001 C CNN
 F 3 "~" H 1800 4950 50  0001 C CNN
 	1    1800 4950
@@
 F 0 "J5" V 1600 5750 50  0000 L CNN
 F 1 "FAN0" V 1700 5850 50  0000 L CNN
-F 2 "Connector_JST:JST_EH_B2B-EH-A_1x02_P2.50mm_Vertical" H 1600 6000 50  0001 C CNN
+F 2 "Connector_JST:JST_XH_B2B-XH-A_1x02_P2.50mm_Vertical" H 1600 6000 50  0001 C CNN
 F 3 "~" H 1600 6000 50  0001 C CNN
 	1    1600 6000
@@
 F 0 "J30" V 4250 4850 50  0000 L CNN
 F 1 "Z-Stop" V 4350 4900 50  0000 L CNN
-F 2 "Connector_JST:JST_EH_B3B-EH-A_1x03_P2.50mm_Vertical" H 4250 5100 50  0001 C CNN
+F 2 "Connector_JST:JST_XH_B3B-XH-A_1x03_P2.50mm_Vertical" H 4250 5100 50  0001 C CNN
 F 3 "~" H 4250 5100 50  0001 C CNN
 	1    4250 5100
@@
 F 0 "J26" V 3750 4850 50  0000 L CNN
 F 1 "Y-Stop" V 3850 4900 50  0000 L CNN
-F 2 "Connector_JST:JST_EH_B3B-EH-A_1x03_P2.50mm_Vertical" H 3750 5100 50  0001 C CNN
+F 2 "Connector_JST:JST_XH_B3B-XH-A_1x03_P2.50mm_Vertical" H 3750 5100 50  0001 C CNN
 F 3 "~" H 3750 5100 50  0001 C CNN
 	1    3750 5100
@@
 F 0 "J23" V 3250 4850 50  0000 L CNN
 F 1 "X-Stop" V 3350 4900 50  0000 L CNN
-F 2 "Connector_JST:JST_EH_B3B-EH-A_1x03_P2.50mm_Vertical" H 3250 5100 50  0001 C CNN
+F 2 "Connector_JST:JST_XH_B3B-XH-A_1x03_P2.50mm_Vertical" H 3250 5100 50  0001 C CNN
 F 3 "~" H 3250 5100 50  0001 C CNN
 	1    3250 5100
@@
 F 0 "J14" V 2350 800 50  0000 L CNN
 F 1 "ZM1" V 2350 950 50  0000 L CNN
-F 2 "Connector_JST:JST_EH_B4B-EH-A_1x04_P2.50mm_Vertical" H 2250 950 50  0001 C CNN
+F 2 "Connector_JST:JST_XH_B4B-XH-A_1x04_P2.50mm_Vertical" H 2250 950 50  0001 C CNN
 F 3 "~" H 2250 950 50  0001 C CNN
 	1    2250 950
@@
 F 0 "J7" V 1850 900 50  0000 R CNN
 F 1 "YM" V 1850 1050 50  0000 R CNN
-F 2 "Connector_JST:JST_EH_B4B-EH-A_1x04_P2.50mm_Vertical" H 1750 950 50  0001 C CNN
+F 2 "Connector_JST:JST_XH_B4B-XH-A_1x04_P2.50mm_Vertical" H 1750 950 50  0001 C CNN
 F 3 "~" H 1750 950 50  0001 C CNN
 	1    1750 950
@@
 F 0 "J21" V 3350 850 50  0000 R CNN
 F 1 "EM0" V 3350 1050 50  0000 R CNN
-F 2 "Connector_JST:JST_EH_B4B-EH-A_1x04_P2.50mm_Vertical" H 3250 950 50  0001 C CNN
+F 2 "Connector_JST:JST_XH_B4B-XH-A_1x04_P2.50mm_Vertical" H 3250 950 50  0001 C CNN
 F 3 "~" H 3250 950 50  0001 C CNN
 	1    3250 950
